File: KiCad/GR_Low_Side_Switch.kicad_pcb (KiCad board)
At the start: 2 copper layers, 99.9 x 100 mm, 202 parts, among them J1 Screw_Terminal_01x03, J10 Conn_01x02, J2 Screw_Terminal_01x02, J3 Screw_Terminal_01x01, J4 Screw_Terminal_01x08, J5 Screw_Terminal_01x08, J6 Screw_Terminal_01x04, J7 Screw_Terminal_01x16, J8 Screw_Terminal_01x08, J9 Screw_Terminal_01x08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

Commit message: Add files via upload
Other:
- board text added: "+5V"
- board text added: "GND"
- board text added: "Rev 1.0"
